File: kicad/no48v/AudioPowerSupply_Acramonics.kicad_sch (KiCad schematic)
At the start: 23 parts, among them J2 Conn_01x04_Pin, T1 12-0-12V, U1 LM7815_TO220, U2 LM7915_TO220

Commit message: Added scripts to generate non 48V version and a PCB and BOM for this
Other:
- removed sheet 48V-Booster
Changed lines of the file:
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@@
-		)
-	)
-	(sheet
-		(at 176.53 60.96)
-		(size 12.7 5.08)
-		(exclude_from_sim no)
-		(in_bom yes)
-		(on_board yes)
-		(dnp no)
-		(fields_autoplaced yes)
-		(stroke
-			(width 0.1524)
-			(type solid)
-		)
-		(fill
-			(color 0 0 0 0)
-		)
-		(property "Sheetname" "48V-Booster"
-			(at 176.53 60.2484 0)
-			(show_name no)
-			(do_not_autoplace no)
-			(effects
-				(font
-					(size 1.27 1.27)
-				)
-				(justify left bottom)
-			)
-		)
-		(property "Sheetfile" "48V-Booster.kicad_sch"
-			(at 176.53 66.6246 0)
-			(show_name no)
-			(do_not_autoplace no)
-			(effects
-				(font
-					(size 1.27 1.27)
-				)
-				(justify left top)
-			)
-		)
-		(instances
-			(project "AudioPowerSupply_Acramonics"
-				(path "/56a175f5-4366-4bc8-b594-267ae81190c5"
-					(page "2")
-				)
-			)
 		)
 	)
